Commit message: Add Pi-side tag EKF, follow controller, and web dashboard
Estimation + control:
- tag_estimator: EKF over the tag's (x,y) in odom, fusing uwb/raw + pan angle
  + odom, with online UWB<->IMU latency calibration -> fused/tag_pose
- nav_controller: latched-goal follow-me. Commits the tag as a point in odom
  and steers to it; HOLDs (freezes the goal, keeps driving to the last trusted
  point) above 10 deg bearing sigma and re-acquires below 7 deg. Broadcasts
  odom -> nav_goal. In bringup behind follow:=true (default off - it drives).

Interfaces: add ActuatorStatus, CommandStatus, DisplayFlag, DriveCommand,
TagEstimate, UwbRaw, WheelState; drop FusedTagPose with the ESP32 telemetry
slim-down.

Web dashboard: static React/Vite SPA over the Foxglove ws-protocol - top-down
2D view of the car, the fused tag estimate, and the committed nav_goal.

Also: serial_bridge/launch/urdf updates, node unit tests, and a doc refresh
(NOTES build log, PROJECT_PLAN, cheat.md). Removes the superseded
hal-command-path spec and the T2 bridge-TX brief.

File: src/follow_me_nodes/urdf/follow_me_car.urdf (robot description, URDF)
Before this commit: robot follow_me_car, 9 links, 8 joints
Links:
- link body_link: geometry visual box size=0.300 0.170 0.070
- link chassis_link: geometry visual box size=0.024 0.056 0.010; visual box size=0.024 0.056 0.010
- link imu_link: geometry visual box size=0.030 0.020 0.010
- link uwb_link: geometry visual box size=0.100 0.020 0.008
Joints:
- joint base_to_front_left_wheel: axis (none) -> 0 0 1; limit (none) -> lower=-0.5236 upper=0.5236 effort=1.0 velocity=7.0; type fixed -> revolute
- joint base_to_front_right_wheel: axis (none) -> 0 0 1; limit (none) -> lower=-0.5236 upper=0.5236 effort=1.0 velocity=7.0; type fixed -> revolute
- joint base_to_imu: origin xyz=-0.100 0 0.053 rpy=0 0 0 -> xyz=-0.110 0 0.125 rpy=0 0 0
- joint base_to_uwb: axis (none) -> 0 0 1; limit (none) -> lower=-0.9599 upper=0.9599 effort=1.0 velocity=0.8727; origin xyz=0.150 0 0.135 rpy=0 0 0 -> xyz=0.090 0 0.130 rpy=0 0 0; type fixed -> revolute
